File: Hardware/eagle/TouchBoxLED/LEDboard_v0.4-R001.brd (EAGLE design)
At the start: 100.3 x 14.7 mm, 13 parts, among them X1 22-23-2021, X2 22-23-2021, X3 22-23-2021

Commit message: cleanup, new screen shot, readme etc
Routing:
- net N$11: track 18.6 -> 19.4 mm
- net N$10: track 9.74 -> 10.5 mm
- net N$7: track 53.8 -> 54.4 mm
- net N$8: vias 0 -> 2
Other:
- outline, holes or cut-outs redrawn
